Commit message: Vacuum Gripper done

File: install/ur5/share/ur5/ur5_bot.urdf (robot description, URDF)
Before this commit: robot ur5, 14 links, 13 joints
Links:
- removed link camera_link_optical
- link vacuum_gripper1: geometry visual cylinder length=0.03 radius=0.005
- link vacuum_gripper2: geometry visual cylinder length=0.03 radius=0.005
- link vacuum_gripper3: geometry visual cylinder length=0.03 radius=0.005
- link vacuum_gripper4: geometry visual cylinder length=0.03 radius=0.005
Joints:
- removed joint camera_optical_joint
- joint gripper_joint1: type fixed -> revolute
- joint gripper_joint2: type fixed -> revolute
- joint gripper_joint3: type fixed -> revolute
- joint gripper_joint4: type fixed -> revolute
- joint shoulder_lift_joint: limit lower=-1.57 upper=1.57 effort=200 velocity=3 -> lower=-6.2832 upper=6.2832 effort=200 velocity=3
- joint wrist_3_joint: limit lower=-6.2832 upper=6.2832 effort=100 velocity=3 -> lower=-6.2832 upper=6.2832 effort=200 velocity=3

File: install/ur5/share/ur5/ur5_rviz_bot.urdf (robot description, URDF)
Before this commit: robot ur5, 8 links, 7 joints
Links:
- added link camera_link, mass 1e-5; collision box size=0.02 0.02 0.02; visual box size=0.02 0.02 0.02
- added link camera_link_optical
- added link vacuum_gripper1, mass 0.0001; visual cylinder length=0.01 radius=0.005
- added link vacuum_gripper2, mass 0.0001; visual cylinder length=0.01 radius=0.005
- added link vacuum_gripper3, mass 0.0001; visual cylinder length=0.01 radius=0.005
- added link vacuum_gripper4, mass 0.0001; visual cylinder length=0.01 radius=0.005
- link base_link: mass 0.50431 -> 4.0
- link forearm_link: mass 2.6854 -> 2.275
- link shoulder_link: mass 1.573 -> 3.7
- link upper_arm_link: mass 4.6689 -> 8.393
- link wrist_1_link: mass 0.54083 -> 1.219
- link wrist_2_link: mass 0.54083 -> 1.219
- link wrist_3_link: mass 0.16482 -> 0.1879
Joints:
- added joint camera_joint: type fixed, parent wrist_3_link, child camera_link, origin xyz=0.04 0.02 0 rpy=0 0 0, axis 0 1 0
- added joint camera_optical_joint: type fixed, parent camera_link, child camera_link_optical, origin xyz=0 0 0 rpy=-1.5708 0 -1.5708
- added joint gripper_joint1: type fixed, parent wrist_3_link, child vacuum_gripper1, origin xyz=0.01 0.04 0 rpy=1.570 0 0, axis 1 0 0, limit lower=0 upper=0 effort=50 velocity=50
- added joint gripper_joint2: type fixed, parent wrist_3_link, child vacuum_gripper2, origin xyz=-0.01 0.04 0 rpy=1.570 0 0, axis 1 0 0, limit lower=0 upper=0 effort=50 velocity=50
- added joint gripper_joint3: type fixed, parent wrist_3_link, child vacuum_gripper3, origin xyz=0 0.04 0.01 rpy=1.570 0 0, axis 1 0 0, limit lower=0 upper=0 effort=50 velocity=50
- added joint gripper_joint4: type fixed, parent wrist_3_link, child vacuum_gripper4, origin xyz=0 0.04 -0.01 rpy=1.570 0 0, axis 1 0 0, limit lower=0 upper=0 effort=50 velocity=50

Commit message: Removed Errors

File: install/ur5/share/ur5/ur5_bot.urdf (robot description, URDF)
Before this commit: robot ur5, 13 links, 12 joints
Links:
- removed link vacuum_gripper2
- removed link vacuum_gripper3
- removed link vacuum_gripper4
- link camera_link: geometry collision box size=0.01 0.01 0.01; visual box size=0.01 0.01 0.01
- link vacuum_gripper1: geometry visual cylinder length=0.015 radius=0.02
Joints:
- removed joint gripper_joint2
- removed joint gripper_joint3
- removed joint gripper_joint4
- joint camera_joint: origin xyz=0.04 0.02 0 rpy=0 0 0 -> xyz=0.03 0.04 0 rpy=0 0 1.508
- joint gripper_joint1: origin xyz=0.01 0.04 0 rpy=1.570 0 0 -> xyz=0 0.04 0 rpy=1.570 0 0
