Commit message: Rviz URDF Updated

File: install/ur5/share/ur5/ur5_rviz_bot.urdf (robot description, URDF)
Before this commit: robot ur5, 14 links, 13 joints
Links:
- removed link camera_link_optical
- removed link vacuum_gripper2
- removed link vacuum_gripper3
- removed link vacuum_gripper4
- link camera_link: geometry collision box size=0.01 0.01 0.01; visual box size=0.01 0.01 0.01
- link vacuum_gripper1: geometry collision box size=0.0 0.0 0.0; visual cylinder length=0.015 radius=0.02
Joints:
- removed joint camera_optical_joint
- removed joint gripper_joint2
- removed joint gripper_joint3
- removed joint gripper_joint4
- joint camera_joint: origin xyz=0.04 0.02 0 rpy=0 0 0 -> xyz=0.03 0.04 0 rpy=0 0 1.508
- joint gripper_joint1: origin xyz=0.01 0.04 0 rpy=1.570 0 0 -> xyz=0 0.04 0 rpy=1.570 0 0; type fixed -> revolute

Commit message: Moveit Obstacle Avoidance Configured

File: install/ur5/share/ur5/ur5_rviz_bot.urdf (robot description, URDF)
Before this commit: robot ur5, 10 links, 9 joints
Links:
- link base_link: geometry collision mesh filename=package://ur5/base_link.stl; visual mesh filename=package://ur5/base_link.stl
- link forearm_link: geometry collision mesh filename=package://ur5/forearm_link.stl; visual mesh filename=package://ur5/forearm_link.stl
- link shoulder_link: geometry collision mesh filename=package://ur5/shoulder_link.stl; visual mesh filename=package://ur5/shoulder_link.stl
- link upper_arm_link: geometry collision mesh filename=package://ur5/upper_arm_link.stl; visual mesh filename=package://ur5/upper_arm_link.stl
- link wrist_1_link: geometry collision mesh filename=package://ur5/wrist_1_link.stl; visual mesh filename=package://ur5/wrist_1_link.stl
- link wrist_2_link: geometry collision mesh filename=package://ur5/wrist_2_link.stl; visual mesh filename=package://ur5/wrist_2_link.stl
- link wrist_3_link: geometry collision mesh filename=package://ur5/wrist_3_link.stl; visual mesh filename=package://ur5/wrist_3_link.stl
